File: bkm-129x-simple-vga.sch (KiCad schematic (older format))
At the start: 55 parts, among them J1 DB15_Female_HighDensity_Mount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, J5 Conn_02x32_Row_Letter_Last, Q1 DTC144EKA, Q2 MMBT3904, SW1 PBH4UEENAGX, U1 ADG1611, U2 THS7374, U3 arduino-nano-v3, U4 74LVC125, U5 MIC3490-3.3

Commit message: Rev. B: Fix THS7374, VGA pin 9, Kicad 5
Parts:
- C1, C10, C11, C12, C2, C3, C4, C5, C6, C9: symbol C -> bkm-129x-simple-vga-rescue:C
- C13, C7, C8: symbol CP -> bkm-129x-simple-vga-rescue:CP
- D1, D2: symbol LED -> bkm-129x-simple-vga-rescue:LED
- J1: symbol DB15_Female_HighDensity_MountingHoles -> bkm-129x-simple-vga-rescue:DB15_Female_HighDensity_MountingHoles
- J5: symbol Conn_02x32_Row_Letter_Last -> bkm-129x-simple-vga-rescue:Conn_02x32_Row_Letter_Last
- Q1: symbol DTC144EKA -> dtc144eka:DTC144EKA
- Q2: symbol Q_NPN_BEC -> bkm-129x-simple-vga-rescue:Q_NPN_BEC
- R1, R10, R11, R12, R13, R14, R15, R16, R18, R19, R2, R20, R21, R22, R23, R24, R25, R26, R27, R28, R3, R32, R33, R34, R4, R5, R6, R7, R8, R9: symbol R -> bkm-129x-simple-vga-rescue:R
- SW1: symbol PBSW_4PDT -> pbsw_4pdt:PBSW_4PDT
- U1: symbol ADG1611 -> adg1611:ADG1611
- U2: symbol THS7374 -> ths7374:THS7374
- U3: symbol arduino-nano-v3 -> arduino-nano-v3:arduino-nano-v3
- U4: symbol 74LVC125 -> bkm-129x-simple-vga-rescue:74LVC125
- U5: symbol MIC3490 -> mic3490:MIC3490
Connections:
- net +3V3: now also U2.9 (BYPASS)
- net GND: no longer J1.9, U2.9 (BYPASS)
- no-connect marks 42 -> 43
